Commit message: feat: Add steerai_sysid and steerai_mpc packages for vehicle dynamics and control, and update URDF joint names.

File: polaris_gem_simulator/gem_simulator/gem_description/urdf/gem.urdf.xacro (robot description, xacro)
@@ -64,10 +64,10 @@
   </link>
   <!-- ***************************************** Set vehicle load point ***************************************** -->
-  <joint name="base_link" type="fixed">
+  <joint name="base_link_joint" type="fixed">
     <origin xyz="0 0 0.44" rpy="0 0 0"/>
     <parent link="base_footprint"/>
     <child link="base_link"/>
   </joint>
-  <joint name="center_link" type="fixed">
+  <joint name="center_link_joint" type="fixed">
     <origin xyz="0.87 0 0.151" rpy="0 0 0"/>
     <parent link="base_link"/>

Commit message: refactor: Remove zero-mass inertial properties from fixed links and update mass/inertia for sonar and bumper links.

File: polaris_gem_simulator/gem_simulator/gem_description/urdf/gem.urdf.xacro (robot description, xacro)
@@ -76,15 +76,4 @@
   <!-- ******************************************* Fixed links below ******************************************* -->
   <link name="chair_link">
-    <inertial>
-      <origin xyz="0 0 0" rpy="0 0 0" />
-      <mass value="0" />
-      <inertia
-        ixx="0"
-        ixy="0"
-        ixz="0"
-        iyy="0"
-        iyz="0"
-        izz="0" />
-    </inertial>
     <visual>
       <origin xyz="0 0 0" rpy="0 0 0" />
@@ -108,15 +97,4 @@
   </joint>
   <link name="door_link">
-    <inertial>
-      <origin xyz="0 0 0" rpy="0 0 0" />
-      <mass value="0" />
-      <inertia
-        ixx="0"
-        ixy="0"
-        ixz="0"
-        iyy="0"
-        iyz="0"
-        izz="0" />
-    </inertial>
     <visual>
       <origin xyz="0 0 0" rpy="0 0 0" />
@@ -140,15 +118,4 @@
   </joint>
   <link name="top_rack_link">
-    <inertial>
-      <origin xyz="0 0 0" rpy="0 0 0" />
-      <mass value="0" />
-      <inertia
-        ixx="0"
-        ixy="0"
-        ixz="0"
-        iyy="0"
-        iyz="0"
-        izz="0" />
-    </inertial>
     <visual>
       <origin xyz="0 0 0" rpy="0 0 0" />
@@ -172,15 +139,4 @@
   </joint>
   <link name="front_rack_link">
-    <inertial>
-      <origin xyz="0 0 0" rpy="0 0 0" />
-      <mass value="0" />
-      <inertia
-        ixx="0."
-        ixy="0"
-        ixz="0"
-        iyy="0"
-        iyz="0"
-        izz="0" />
-    </inertial>
     <visual>
       <origin xyz="0 0 0" rpy="0 0 0" />
@@ -204,15 +160,4 @@
   </joint>
   <link name="rear_rack_link">
-    <inertial>
-      <origin xyz="0 0 0" rpy="0 0 0" />
-      <mass value="0" />
-      <inertia
-        ixx="0"
-        ixy="0"
-        ixz="0"
-        iyy="0"
-        iyz="0"
-        izz="0" />
-    </inertial>
     <visual>
       <origin xyz="0 0 0" rpy="0 0 0" />
@@ -236,15 +181,4 @@
   </joint>
   <link name="front_right_head_light_link">
-    <inertial>
-      <origin xyz="0 0 0" rpy="0 0 0" />
-      <mass value="0" />
-      <inertia
-        ixx="0"
-        ixy="0"
-        ixz="0"
-        iyy="0"
-        iyz="0"
-        izz="0" />
-    </inertial>
     <visual>
       <origin xyz="0 0 0" rpy="0 0 0" />
@@ -268,15 +202,4 @@
   </joint>
   <link name="front_left_head_light_link">
-    <inertial>
-      <origin xyz="0 0 0" rpy="0 0 0" />
-      <mass value="0" />
-      <inertia
-        ixx="0"
-        ixy="0"
-        ixz="0"
-        iyy="0"
-        iyz="0"
-        izz="0" />
-    </inertial>
     <visual>
       <origin xyz="0 0 0" rpy="0 0 0" />
@@ -300,15 +223,4 @@
   </joint>
   <link name="front_right_turn_light_link">
-    <inertial>
-      <origin xyz="0 0 0" rpy="0 0 0" />
-      <mass value="0" />
-      <inertia
-        ixx="0"
-        ixy="0"
-        ixz="0"
-        iyy="0"
-        iyz="0"
-        izz="0" />
-    </inertial>
     <visual>
       <origin xyz="0 0 0" rpy="0 0 0" />
@@ -332,15 +244,4 @@
   </joint>
   <link name="front_left_turn_light_link">
-    <inertial>
-      <origin xyz="0 0 0" rpy="0 0 0" />
-      <mass value="0" />
-      <inertia
-        ixx="0"
-        ixy="0"
-        ixz="0"
-        iyy="0"
-        iyz="0"
-        izz="0" />
-    </inertial>
     <visual>
       <origin xyz="0 0 0" rpy="0 0 0" />
@@ -364,15 +265,4 @@
   </joint>
   <link name="rear_right_light_link">
-    <inertial>
-      <origin xyz="0 0 0" rpy="0 0 0" />
-      <mass value="0" />
-      <inertia
-        ixx="0"
-        ixy="0"
-        ixz="0"
-        iyy="0"
-        iyz="0"
-        izz="0" />
-    </inertial>
     <visual>
       <origin xyz="0 0 0" rpy="0 0 0" />
@@ -396,15 +286,4 @@
   </joint>
   <link name="rear_left_light_link">
-    <inertial>
-      <origin xyz="0 0 0" rpy="0 0 0" />
-      <mass value="0" />
-      <inertia
-        ixx="0"
-        ixy="0"
-        ixz="0"
-        iyy="0"
-        iyz="0"
-        izz="0" />
-    </inertial>
     <visual>
       <origin xyz="0 0 0" rpy="0 0 0" />
@@ -428,15 +307,4 @@
   </joint>
   <link name="rear_left_stop_light_link">
-    <inertial>
-      <origin xyz="0 0 0" rpy="0 0 0" />
-      <mass value="0" />
-      <inertia
-        ixx="0"
-        ixy="0"
-        ixz="0"
-        iyy="0"
-        iyz="0"
-        izz="0" />
-    </inertial>
     <visual>
       <origin xyz="0 0 0" rpy="0 0 0" />
@@ -460,15 +328,4 @@
   </joint>
   <link name="rear_right_stop_light_link">
-    <inertial>
-      <origin xyz="0 0 0" rpy="0 0 0" />
-      <mass value="0" />
-      <inertia
-        ixx="0"
-        ixy="0"
-        ixz="0"
-        iyy="0"
-        iyz="0"
-        izz="0" />
-    </inertial>
     <visual>
       <origin xyz="0 0 0" rpy="0 0 0" />
@@ -492,15 +349,4 @@
   </joint>
   <link name="right_blue_outer_link">
-    <inertial>
-      <origin xyz="0 0 0" rpy="0 0 0" />
-      <mass value="0" />
-      <inertia
-        ixx="0"
-        ixy="0"
-        ixz="0"
-        iyy="0"
-        iyz="0"
-        izz="0" />
-    </inertial>
     <visual>
       <origin xyz="0 0 0" rpy="0 0 0" />
@@ -524,15 +370,4 @@
   </joint>
   <link name="right_I_link">
-    <inertial>
-      <origin xyz="0 0 0" rpy="0 0 0" />
-      <mass value="0" />
-      <inertia
-        ixx="0"
-        ixy="0"
-        ixz="0"
-        iyy="0"
-        iyz="0"
-        izz="0" />
-    </inertial>
     <visual>
       <origin xyz="0 0 0" rpy="0 0 0" />
@@ -556,15 +391,4 @@
   </joint>
   <link name="left_blue_outer_link">
-    <inertial>
-      <origin xyz="0 0 0" rpy="0 0 0" />
-      <mass value="0" />
-      <inertia
-        ixx="0"
-        ixy="0"
-        ixz="0"
-        iyy="0"
-        iyz="0"
-        izz="0" />
-    </inertial>
     <visual>
       <origin xyz="0 0 0" rpy="0 0 0" />
@@ -588,15 +412,4 @@
   </joint>
   <link name="left_I_link">
-    <inertial>
-      <origin xyz="0 0 0" rpy="0 0 0" />
-      <mass value="0" />
-      <inertia
-        ixx="0"
-        ixy="0"
-        ixz="0"
-        iyy="0"
-        iyz="0"
-        izz="0" />
-    </inertial>
     <visual>
       <origin xyz="0 0 0" rpy="0 0 0" />
@@ -620,15 +433,4 @@
   </joint>
   <link name="right_antenna_link">
-    <inertial>
-      <origin xyz="0 0 0" rpy="0 0 0" />
-      <mass value="0" />
-      <inertia
-        ixx="0"
-        ixy="0"
-        ixz="0"
-        iyy="0"
-        iyz="0"
-        izz="0" />
-    </inertial>
     <visual>
       <origin xyz="0 0 0" rpy="0 0 0" />
@@ -652,15 +454,4 @@
   </joint>
   <link name="left_antenna_link">
-    <inertial>
-      <origin xyz="0 0 0" rpy="0 0 0" />
-      <mass value="0" />
-      <inertia
-        ixx="0"
-        ixy="0"
-        ixz="0"
-        iyy="0"
-        iyz="0"
-        izz="0" />
-    </inertial>
     <visual>
       <origin xyz="0 0 0" rpy="0 0 0" />
@@ -684,15 +475,4 @@
   </joint>
   <link name="rear_left_emergency_button_link">
-    <inertial>
-      <origin xyz="0 0 0" rpy="0 0 0" />
-      <mass value="0" />
-      <inertia
-        ixx="0"
-        ixy="0"
-        ixz="0"
-        iyy="0"
-        iyz="0"
-        izz="0" />
-    </inertial>
     <visual>
       <origin xyz="0 0 0" rpy="0 0 0" />
@@ -716,15 +496,4 @@
   </joint>
   <link name="rear_right_emergency_button_link">
-    <inertial>
-      <origin xyz="0 0 0" rpy="0 0 0" />
-      <mass value="0" />
-      <inertia
-        ixx="0"
-        ixy="0"
-        ixz="0"
-        iyy="0"
-        iyz="0"
-        izz="0" />
-    </inertial>
     <visual>
       <origin xyz="0 0 0" rpy="0 0 0" />
@@ -748,15 +517,4 @@
   </joint>
   <link name="front_left_emergency_button_link">
-    <inertial>
-      <origin xyz="0 0 0" rpy="0 0 0" />
-      <mass value="0" />
-      <inertia
-        ixx="0"
-        ixy="0"
-        ixz="0"
-        iyy="0"
-        iyz="0"
-        izz="0" />
-    </inertial>
     <visual>
       <origin xyz="0 0 0" rpy="0 0 0" />
@@ -780,15 +538,4 @@
   </joint>
   <link name="front_right_emergency_button_link">
-    <inertial>
-      <origin xyz="0 0 0" rpy="0 0 0" />
-      <mass value="0" />
-      <inertia
-        ixx="0"
-        ixy="0"
-        ixz="0"
-        iyy="0"
-        iyz="0"
-        izz="0" />
-    </inertial>
     <visual>
       <origin xyz="0 0 0" rpy="0 0 0" />
@@ -812,9 +559,4 @@
   </joint>
   <link name="rear_light_bar_link">
-    <inertial>
-      <origin xyz="0 0 0" rpy="0 0 0" />
-      <mass value="0" />
-      <inertia ixx="0" ixy="0" ixz="0" iyy="0" iyz="0" izz="0" />
-    </inertial>
     <visual>
       <origin xyz="0 0 0" rpy="0 0 0" />
@@ -1059,7 +801,7 @@
     </visual>
     <inertial>
-      <mass value="1e-5" />
-      <origin xyz="0 0 0" rpy="0 0 0"/>
-      <inertia ixx="1e-6" ixy="0" ixz="0" iyy="1e-6" iyz="0" izz="1e-6" />
+      <mass value="0.1" />
+      <origin xyz="0 0 0" rpy="0 0 0"/>
+      <inertia ixx="0.001" ixy="0" ixz="0" iyy="0.001" iyz="0" izz="0.001" />
     </inertial>
   </link>
@@ -1159,10 +901,9 @@
   </joint>
   <!-- ************************* Front Sonar ************************* -->
-  <!--
   <link name="front_sonar_link">
     <inertial>
-      <mass value="0.001" />
-      <origin xyz="0 0 0" rpy="0 0 0" />
-      <inertia ixx="0.000000017" ixy="0" ixz="0" iyy="0.000000017" iyz="0" izz="0.000000017" />
+      <mass value="0.1" />
+      <origin xyz="0 0 0" rpy="0 0 0" />
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